File: tvca_controller/tvca_controller.kicad_pcb (KiCad board)
At the start: 2 copper layers, 55 parts, among them J1 Programming Header, J2 PT 1,5/ 4-5,0-H, J3 4DB-P108-02, J4 PT 1,5/ 4-5,0-H, J5 4DB-P108-02, J6 PT 1,5/ 4-5,0-H, J7 4DB-P108-02, J9 4DB-P108-02, U1 PIC18F26K83, U2 MCP2562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

Commit message: Fix units/R-sense calculation
Parts:
- C1, C2: value 27 pF -> 27pF
- C10, C11: value 270 uF -> 270uF
- C12, C13, C4, C5: value 0.1 uF -> 0.1uF
- C3: value 10 uF -> 10uF
- C6, C7: value 10 nF -> 10nF
- C8, C9: value 100 nF -> 100nF
- F1: value 350 mA -> 350mA
- F2, F4: value 25 A -> 25A
- R1, R18, R19: value 10 K -> 10k
- R10, R11, R14, R15, R16, R17, R5, R6: value 1 K -> 1k
- R2: value 200 mR 1% -> 200mR 1%
- R7, R8: value 400 R -> 866R 1%
- R9: value 330 R -> 330R
Changed lines of the file:
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@@
         (effects (font (size 1 1) (thickness 0.15)))
     )
-    (fp_text value "1 K" (at 0 1.65) (layer "F.Fab")
+    (fp_text value "1k" (at 0 1.65) (layer "F.Fab")
         (effects (font (size 1 1) (thickness 0.15)))
     )
@@
         (effects (font (size 1 1) (thickness 0.15)))
     )
-    (fp_text value "270 uF" (at 2.5 7.5) (layer "F.Fab")
+    (fp_text value "270uF" (at 2.5 7.5) (layer "F.Fab")
         (effects (font (size 1 1) (thickness 0.15)))
     )
@@
         (effects (font (size 1 1) (thickness 0.15)))
     )
-    (fp_text value "1 K" (at 0 1.65) (layer "F.Fab")
+    (fp_text value "1k" (at 0 1.65) (layer "F.Fab")
         (effects (font (size 1 1) (thickness 0.15)))
     )
@@
         (effects (font (size 1 1) (thickness 0.1)))
     )
-    (fp_text value "25 A" (at 0 13.74 unlocked) (layer "F.Fab")
+    (fp_text value "25A" (at 0 13.74 unlocked) (layer "F.Fab")
         (effects (font (size 1 1) (thickness 0.15)))
     )
@@
         (effects (font (size 1 1) (thickness 0.15)))
     )
-    (fp_text value "10 K" (at 0 1.65) (layer "F.Fab")
+    (fp_text value "10k" (at 0 1.65) (layer "F.Fab")
         (effects (font (size 1 1) (thickness 0.15)))
     )
@@
         (effects (font (size 1 1) (thickness 0.15)))
     )
-    (fp_text value "0.1 uF" (at 0 1.68) (layer "F.Fab")
+    (fp_text value "0.1uF" (at 0 1.68) (layer "F.Fab")
         (effects (font (size 1 1) (thickness 0.15)))
     )
@@
         (effects (font (size 1 1) (thickness 0.1)))
     )
-    (fp_text value "25 A" (at 0 13.74 unlocked) (layer "F.Fab")
+    (fp_text value "25A" (at 0 13.74 unlocked) (layer "F.Fab")
         (effects (font (size 1 1) (thickness 0.15)))
     )
@@
         (effects (font (size 1 1) (thickness 0.15)))
     )
-    (fp_text value "330 R" (at 0 1.65) (layer "F.Fab")
+    (fp_text value "330R" (at 0 1.65) (layer "F.Fab")
         (effects (font (size 1 1) (thickness 0.15)))
     )
@@
         (effects (font (size 1 1) (thickness 0.15)))
     )
-    (fp_text value "270 uF" (at 2.5 7.5) (layer "F.Fab")
+    (fp_text value "270uF" (at 2.5 7.5) (layer "F.Fab")
         (effects (font (size 1 1) (thickness 0.15)))
     )
@@
         (effects (font (size 1 1) (thickness 0.15)))
     )
-    (fp_text value "1 K" (at 0 1.65) (layer "F.Fab")
+    (fp_text value "1k" (at 0 1.65) (layer "F.Fab")
         (effects (font (size 1 1) (thickness 0.15)))
     )
@@
         (effects (font (size 1 1) (thickness 0.15)))
     )
-    (fp_text value "1 K" (at 0 1.65) (layer "F.Fab")
+    (fp_text value "1k" (at 0 1.65) (layer "F.Fab")
         (effects (font (size 1 1) (thickness 0.15)))
     )
@@
         (effects (font (size 1 1) (thickness 0.15)))
     )
-    (fp_text value "1 K" (at 0 1.65) (layer "F.Fab")
+    (fp_text value "1k" (at 0 1.65) (layer "F.Fab")
         (effects (font (size 1 1) (thickness 0.15)))
     )
@@
         (effects (font (size 1 1) (thickness 0.15)))
     )
-    (fp_text value "1 K" (at 0 1.65) (layer "F.Fab")
+    (fp_text value "1k" (at 0 1.65) (layer "F.Fab")
         (effects (font (size 1 1) (thickness 0.15)))
     )
@@
         (effects (font (size 1 1) (thickness 0.15)))
     )
-    (fp_text value "27 pF" (at 0 1.68) (layer "F.Fab")
+    (fp_text value "27pF" (at 0 1.68) (layer "F.Fab")
         (effects (font (size 1 1) (thickness 0.15)))
     )
@@
         (effects (font (size 1 1) (thickness 0.15)))
     )
-    (fp_text value "400 R" (at 0 1.65 90) (layer "F.Fab")
+    (fp_text value "866R 1%" (at 0 1.65 90) (layer "F.Fab")
         (effects (font (size 1 1) (thickness 0.15)))
     )
@@
         (effects (font (size 1 1) (thickness 0.15)))
     )
-    (fp_text value "400 R" (at 0 1.65) (layer "F.Fab")
+    (fp_text value "866R 1%" (at 0 1.65) (layer "F.Fab")
         (effects (font (size 1 1) (thickness 0.15)))
     )
@@
         (effects (font (size 1 1) (thickness 0.15)))
     )
-    (fp_text value "10 K" (at 0 1.65) (layer "F.Fab")
+    (fp_text value "10k" (at 0 1.65) (layer "F.Fab")
         (effects (font (size 1 1) (thickness 0.15)))
     )
@@
         (effects (font (size 1 1) (thickness 0.15)))
     )
-    (fp_text value "27 pF" (at 0 1.68) (layer "F.Fab")
+    (fp_text value "27pF" (at 0 1.68) (layer "F.Fab")
         (effects (font (size 1 1) (thickness 0.15)))
     )
@@
         (effects (font (size 1 1) (thickness 0.15)))
     )
-    (fp_text value "0.1 uF" (at 0 1.68) (layer "F.Fab")
+    (fp_text value "0.1uF" (at 0 1.68) (layer "F.Fab")
         (effects (font (size 1 1) (thickness 0.15)))
     )
@@
         (effects (font (size 1 1) (thickness 0.15)))
     )
-    (fp_text value "0.1 uF" (at 0 1.68) (layer "F.Fab")
+    (fp_text value "0.1uF" (at 0 1.68) (layer "F.Fab")
         (effects (font (size 1 1) (thickness 0.15)))
     )
@@
         (effects (font (size 1 1) (thickness 0.15)))
     )
-    (fp_text value "1 K" (at 0 1.65) (layer "F.Fab")
+    (fp_text value "1k" (at 0 1.65) (layer "F.Fab")
         (effects (font (size 1 1) (thickness 0.15)))
     )
@@
         (effects (font (size 1 1) (thickness 0.15)))
     )
-    (fp_text value "100 nF" (at 0 1.68) (layer "F.Fab")
+    (fp_text value "100nF" (at 0 1.68) (layer "F.Fab")
         (effects (font (size 1 1) (thickness 0.15)))
     )
@@
         (effects (font (size 1 1) (thickness 0.15)))
     )
-    (fp_text value "10 nF" (at 0 1.68 90) (layer "F.Fab")
+    (fp_text value "10nF" (at 0 1.68 90) (layer "F.Fab")
         (effects (font (size 1 1) (thickness 0.15)))
     )
@@
         (effects (font (size 1 1) (thickness 0.15)))
     )
-    (fp_text value "200 mR 1%" (at 0 1.65) (layer "F.Fab")
+    (fp_text value "200mR 1%" (at 0 1.65) (layer "F.Fab")
         (effects (font (size 1 1) (thickness 0.15)))
     )
@@
         (effects (font (size 1 1) (thickness 0.15)))
     )
-    (fp_text value "350 mA" (at 0 1.82) (layer "F.Fab")
+    (fp_text value "350mA" (at 0 1.82) (layer "F.Fab")
         (effects (font (size 1 1) (thickness 0.15)))
     )
@@
         (effects (font (size 1 1) (thickness 0.15)))
     )
-    (fp_text value "0.1 uF" (at 0 1.68) (layer "F.Fab")
+    (fp_text value "0.1uF" (at 0 1.68) (layer "F.Fab")
         (effects (font (size 1 1) (thickness 0.15)))
     )
@@
         (effects (font (size 1 1) (thickness 0.15)))
     )
-    (fp_text value "10 nF" (at 0 1.68) (layer "F.Fab")
+    (fp_text value "10nF" (at 0 1.68) (layer "F.Fab")
         (effects (font (size 1 1) (thickness 0.15)))
     )
@@
         (effects (font (size 1 1) (thickness 0.15)))
     )
-    (fp_text value "10 K" (at 0 1.65) (layer "F.Fab")
+    (fp_text value "10k" (at 0 1.65) (layer "F.Fab")
         (effects (font (size 1 1) (thickness 0.15)))
     )
@@
         (effects (font (size 1 1) (thickness 0.15)))
     )
-    (fp_text value "10 uF" (at 0 1.68) (layer "F.Fab")
+    (fp_text value "10uF" (at 0 1.68) (layer "F.Fab")
         (effects (font (size 1 1) (thickness 0.15)))
     )
@@
         (effects (font (size 1 1) (thickness 0.15)))
     )
-    (fp_text value "1 K" (at 0 1.65) (layer "F.Fab")
+    (fp_text value "1k" (at 0 1.65) (layer "F.Fab")
         (effects (font (size 1 1) (thickness 0.15)))
     )
@@
         (effects (font (size 1 1) (thickness 0.15)))
     )
-    (fp_text value "100 nF" (at 0 1.68) (layer "F.Fab")
+    (fp_text value "100nF" (at 0 1.68) (layer "F.Fab")
         (effects (font (size 1 1) (thickness 0.15)))
     )

Commit message: New PCB layout
Parts:
- C10, C11, C12, C13, C5, F1, J4, J6, R10, R11, R12, R13, R14, R15, R16, R17, R2, R3, R4, R5, R6, TP9, U2, U3: moved to B.Cu
- moved Y1 96.2 mm to (151.7, 55.3), turned to 180 degrees
- moved U3 93.4 mm to (151.8, 63.5)
- moved R1 91.9 mm to (161.9, 54.8), turned to -90 degrees
- moved R2 91.0 mm to (146.7, 63.5), turned to 180 degrees
- moved C2 87.4 mm to (141.6, 54.8), turned to -90 degrees
- moved C4 85.1 mm to (167.0, 54.8), turned to -90 degrees
- moved J1 83.9 mm to (164.6, 58.4), turned to -90 degrees
- moved C5 82.0 mm to (156.8, 63.5)
- moved R9 81.2 mm to (159.4, 72.4)
- moved F1 80.1 mm to (141.6, 63.5)
- moved J2 79.9 mm to (126.4, 54.6), turned to -90 degrees
- moved TP9 79.2 mm to (140.3, 59.7), turned to 180 degrees
- moved C1 78.7 mm to (156.8, 54.8), turned to -90 degrees
- moved C3 78.0 mm to (141.6, 68.6), turned to 90 degrees
- moved U1 76.5 mm to (152.4, 64.5), turned to -90 degrees
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Connections:
- J5 pad 1: /Motor_1/OUT_1 -> /Motor_1/OUT_2
- J5 pad 2: /Motor_1/OUT_2 -> /Motor_1/OUT_1
- J7 pad 1: /Motor_2/OUT_1 -> /Motor_2/OUT_2
- J7 pad 2: /Motor_2/OUT_2 -> /Motor_2/OUT_1

Commit message: address a set of comments
Parts:
- C12, C13, TP9: moved to F.Cu
- moved TP9 33.4 mm to (173.4, 54.6), turned to 0 degrees
- moved C4 24.5 mm to (149.9, 72.4), turned to 180 degrees
- moved TP7 13.1 mm to (122.6, 62.9)
- moved TP8 13.1 mm to (122.6, 68.0)
- moved TP6 13.1 mm to (122.6, 73.0)
- moved TP5 13.1 mm to (122.6, 57.8)
- moved C5 8.52 mm to (149.2, 67.3), turned to 180 degrees
- moved C7 6.35 mm to (139.1, 133.3), turned to 180 degrees
- moved R8 5.68 mm to (139.1, 141.0), turned to 0 degrees
- moved J2 5.47 mm to (130.8, 57.8)
- moved R2 4.57 mm to (149.2, 59.7)
- moved R11 4.44 mm to (135.9, 135.9)
- moved R17 4.44 mm to (135.9, 141.0)
- moved C12 3.82 mm to (131.4, 80.0), turned to 0 degrees
- moved R19 3.81 mm to (139.1, 137.2)
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
Commit message: finalize layout
Parts:
- removed TP5: 5V, TestPoint:TestPoint_THTPad_2.5x2.5mm_Drill1.2mm
- removed TP6: GND, TestPoint:TestPoint_THTPad_2.5x2.5mm_Drill1.2mm
- removed TP7: CANH, TestPoint:TestPoint_THTPad_2.5x2.5mm_Drill1.2mm
- removed TP8: CANL, TestPoint:TestPoint_THTPad_2.5x2.5mm_Drill1.2mm
- added H1: Mount, MountingHole:MountingHole_3.2mm_M3_Pad, F.Cu at (114.3, 101.0)
- added H2: Mount, MountingHole:MountingHole_3.2mm_M3_Pad, F.Cu at (189.9, 101.0)
- added H3: Mount, MountingHole:MountingHole_3.2mm_M3_Pad, F.Cu at (189.9, 152.4)
- added H4: Mount, MountingHole:MountingHole_3.2mm_M3_Pad, F.Cu at (114.3, 153.0)
- added TP1: TestPoint, TestPoint:TestPoint_THTPad_2.5x2.5mm_Drill1.2mm, F.Cu at (192.5, 140.7)
- added TP2: TestPoint, TestPoint:TestPoint_THTPad_2.5x2.5mm_Drill1.2mm, F.Cu at (112.3, 139.7)
- C1, C12, C13, C2, C3, C6, C7, J1, R18, R19, R7, R8, Y1: moved to B.Cu
- C10, C11, J4, J6, R10, R11, R12, R13, R14, R15, R16, R17, R3, R4, R5, R6: moved to F.Cu
- moved J2 93.8 mm to (144.8, 150.5), turned to 0 degrees
- moved C2 86.0 mm to (145.9, 140.7), turned to 180 degrees
- moved Y1 75.6 mm to (145.9, 130.6), turned to -90 degrees
- moved C1 71.5 mm to (145.9, 125.5), turned to 180 degrees
- moved U2 69.7 mm to (152.8, 137.4), turned to -90 degrees
- moved R1 68.3 mm to (145.3, 121.0)
- moved U1 66.1 mm to (152.9, 130.6), turned to 0 degrees
- moved R2 65.4 mm to (156.1, 124.7), turned to 90 degrees
- moved C3 64.7 mm to (152.8, 132.3), turned to 180 degrees
- moved C4 61.9 mm to (160.9, 133.3), turned to -90 degrees
- moved U3 61.6 mm to (152.9, 125.0), turned to -90 degrees
- moved F1 58.4 mm to (156.1, 119.9), turned to -90 degrees
- moved C5 57.5 mm to (149.9, 124.8), turned to 90 degrees
- moved C13 51.6 mm to (184.7, 125.7), turned to -90 degrees
- moved J1 49.5 mm to (157.5, 107.4), turned to 180 degrees
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
Commit message: add final layout and edge cuts
Parts:
- C1, C2: moved to F.Cu
- moved C2 24.6 mm to (140.2, 116.8), turned to -90 degrees
- moved J3 23.7 mm to (172.5, 85.6)
- moved TP1 23.5 mm to (187.2, 117.9)
- moved H1 23.2 mm to (108.5, 78.5)
- moved H4 23.2 mm to (108.5, 130.6)
- moved TP3 23.0 mm to (156.5, 76.7)
- moved H2 22.9 mm to (185.7, 78.5)
- moved J2 22.8 mm to (139.7, 128.3)
- moved J9 22.7 mm to (129.0, 85.6)
- moved C10 22.4 mm to (165.1, 101.6)
- moved F1 22.4 mm to (151.1, 98.1)
- moved F4 22.4 mm to (134.4, 100.1)
- moved R1 22.4 mm to (140.2, 99.2)
- moved R10 22.4 mm to (161.3, 109.7)
- moved R14 22.4 mm to (161.3, 115.8)
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- renumbered TP9 to TP3
Other:
- board outline added: 84.3 x 59.2 mm

Commit message: High power routing
Parts:
- J1: moved to F.Cu
- moved F1 12.9 mm to (146.1, 110.0), turned to 90 degrees
- moved R18 12.4 mm to (161.2, 112.3), turned to 0 degrees
- moved R19 10.7 mm to (132.6, 112.3), turned to 180 degrees
- moved R10 10.2 mm to (161.1, 119.9)
- moved J1 10.2 mm to (140.7, 86.0), turned to 0 degrees
- moved R7 8.85 mm to (161.2, 115.3), turned to 180 degrees
- moved C5 7.78 mm to (152.3, 105.1), turned to -90 degrees
- moved D1 7.37 mm to (154.2, 90.0), turned to 90 degrees
- moved R8 6.88 mm to (132.6, 115.3), turned to 0 degrees
- moved C6 6.76 mm to (161.2, 118.4), turned to 0 degrees
- moved R2 5.46 mm to (146.1, 105.2), turned to -90 degrees
- moved R14 5.08 mm to (161.1, 110.7)
- moved C7 4.85 mm to (132.6, 118.4), turned to 180 degrees
- moved C3 4.32 mm to (152.0, 109.9)
- moved U2 4.32 mm to (152.0, 115.0)
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Routing:
- net /Motor_2/OUT_1: track 0.00 -> 13.6 mm, vias 0 -> 2
- net /Motor_2/OUT_2: track 0.00 -> 12.7 mm, vias 0 -> 2
- net /Motor_1/OUT_1: track 0.00 -> 12.7 mm, vias 0 -> 2
- net /Motor_1/OUT_2: track 0.00 -> 11.5 mm, vias 0 -> 2
- net /Motor_2/POWER: vias 0 -> 3
- net /Motor_1/POWER: vias 0 -> 3
- added copper zone on B.Cu, net /Motor_1/OUT_1
- added copper zone on F.Cu, net /Motor_1/OUT_1
- added copper zone on B.Cu, net /Motor_1/OUT_2
- added copper zone on F.Cu, net /Motor_1/OUT_2
- added copper zone on B.Cu, net /Motor_1/POWER
- added copper zone on F.Cu, net /Motor_1/POWER
- added copper zone on B.Cu, net /Motor_2/OUT_1
- added copper zone on F.Cu, net /Motor_2/OUT_1
- added copper zone on B.Cu, net /Motor_2/OUT_2
- added copper zone on F.Cu, net /Motor_2/OUT_2
- added copper zone on B.Cu, net /Motor_2/POWER
- added copper zone on F.Cu, net /Motor_2/POWER
- added copper zone on B.Cu, net GND
- added copper zone on F.Cu, net GND
- added copper zone on B.Cu, net Net-(J3-Pin_1)
- added copper zone on F.Cu, net Net-(J3-Pin_1)
- added copper zone on B.Cu, net Net-(J9-Pin_1)
- added copper zone on F.Cu, net Net-(J9-Pin_1)

Commit message: small fix
Parts:
- moved C9 0.29 mm to (122.6, 109.7)
Routing:
- net /Motor_2/OUT_1: track 13.6 -> 19.5 mm
- net /Motor_1/OUT_2: track 11.5 -> 16.4 mm
- net /Motor_2/POWER: track 0.00 -> 4.63 mm
- net /Motor_1/POWER: track 0.00 -> 4.63 mm
- net /Motor_1/OUT_1: track 12.7 -> 16.5 mm
- net /Motor_2/OUT_2: track 12.7 -> 16.4 mm
Changed lines of the file:
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@@
   )
   (footprint "Capacitor_SMD:C_0805_2012Metric_Pad1.18x1.45mm_HandSolder" (layer "F.Cu")
-    (at 122.555 110.017 180)
+    (at 122.555 109.728 180)
     (descr "Capacitor SMD 0805 (2012 Metric), square (rectangular) end terminal, IPC_7351 nominal with elongated pad for handsoldering. (Body size source: IPC-SM-782 page 76, https://www.pcb-3d.com/wordpress/wp-content/uploads/ipc-sm-782a_amendment_1_and_2.pdf, https://docs.google.com/spreadsheets/d/1BsfQQcO9C6DZCsRaXUlFlo91Tg2WpOkGARC1WS5S8t0/edit?usp=sharing), generated with kicad-footprint-generator")
     (tags "capacitor handsolder")
@@
   (gr_arc (start 189.23 130.556) (mid 188.188472 133.070472) (end 185.674 134.112)
     (stroke (width 0.1) (type default)) (layer "Edge.Cuts"))
-  (via (at 168.656 112.141) (size 0.8) (drill 0.4) (layers "F.Cu" "B.Cu") (net 21))
-  (via (at 169.926 112.141) (size 0.8) (drill 0.4) (layers "F.Cu" "B.Cu") (net 21))
-  (via (at 168.656 118.491) (size 0.8) (drill 0.4) (layers "F.Cu" "B.Cu") (net 21))
-  (via (at 125.73 112.141) (size 0.8) (drill 0.4) (layers "F.Cu" "B.Cu") (net 22))
-  (via (at 124.46 112.141) (size 0.8) (drill 0.4) (layers "F.Cu" "B.Cu") (net 22))
-  (via (at 124.46 118.491) (size 0.8) (drill 0.4) (layers "F.Cu" "B.Cu") (net 22))
-  (segment (start 172.466 112.776) (end 172.466 112.141) (width 0.635) (layer "F.Cu") (net 43))
+  (segment (start 169.926 112.776) (end 169.926 111.252) (width 0.635) (layer "F.Cu") (net 21))
+  (segment (start 168.656 117.926) (end 168.656 119.507) (width 0.635) (layer "F.Cu") (net 21))
+  (segment (start 168.656 112.776) (end 168.656 111.252) (width 0.635) (layer "F.Cu") (net 21))
+  (via (at 168.656 111.252) (size 0.8) (drill 0.4) (layers "F.Cu" "B.Cu") (net 21))
+  (via (at 169.926 111.252) (size 0.8) (drill 0.4) (layers "F.Cu" "B.Cu") (net 21))
+  (via (at 168.656 119.507) (size 0.8) (drill 0.4) (layers "F.Cu" "B.Cu") (net 21))
+  (segment (start 124.46 117.926) (end 124.46 119.507) (width 0.635) (layer "F.Cu") (net 22))
+  (segment (start 124.46 112.776) (end 124.46 111.252) (width 0.635) (layer "F.Cu") (net 22))
+  (segment (start 125.73 112.776) (end 125.73 111.252) (width 0.635) (layer "F.Cu") (net 22))
+  (via (at 125.73 111.252) (size 0.8) (drill 0.4) (layers "F.Cu" "B.Cu") (net 22))
+  (via (at 124.46 111.252) (size 0.8) (drill 0.4) (layers "F.Cu" "B.Cu") (net 22))
+  (via (at 124.46 119.507) (size 0.8) (drill 0.4) (layers "F.Cu" "B.Cu") (net 22))
+  (segment (start 172.466 112.776) (end 172.466 111.252) (width 0.635) (layer "F.Cu") (net 43))
+  (segment (start 172.466 117.926) (end 172.466 119.507) (width 0.635) (layer "F.Cu") (net 43))
   (segment (start 172.466 112.776) (end 172.466 117.926) (width 0.635) (layer "F.Cu") (net 43))
-  (segment (start 172.466 118.491) (end 172.466 117.926) (width 0.635) (layer "F.Cu") (net 43))
-  (via (at 172.466 118.491) (size 0.8) (drill 0.4) (layers "F.Cu" "B.Cu") (net 43))
-  (via (at 172.466 112.141) (size 0.8) (drill 0.4) (layers "F.Cu" "B.Cu") (net 43))
-  (segment (start 172.466 112.141) (end 172.466 118.491) (width 0.635) (layer "B.Cu") (net 43))
+  (via (at 172.466 119.507) (size 0.8) (drill 0.4) (layers "F.Cu" "B.Cu") (net 43))
+  (via (at 172.466 111.252) (size 0.8) (drill 0.4) (layers "F.Cu" "B.Cu") (net 43))
+  (segment (start 172.466 111.252) (end 172.466 119.507) (width 0.635) (layer "B.Cu") (net 43))
   (segment (start 166.116 112.776) (end 166.116 117.926) (width 0.635) (layer "F.Cu") (net 44))
-  (via (at 166.116 112.141) (size 0.8) (drill 0.4) (layers "F.Cu" "B.Cu") (net 44))
-  (via (at 166.116 118.491) (size 0.8) (drill 0.4) (layers "F.Cu" "B.Cu") (net 44))
-  (segment (start 166.116 112.141) (end 166.116 118.491) (width 0.635) (layer "B.Cu") (net 44))
-  (segment (start 128.27 118.491) (end 128.27 117.926) (width 0.635) (layer "F.Cu") (net 45))
-  (segment (start 128.27 112.776) (end 128.27 112.268) (width 0.635) (layer "F.Cu") (net 45))
-  (segment (start 128.27 112.268) (end 128.27 118.491) (width 0.635) (layer "F.Cu") (net 45))
-  (via (at 128.27 118.491) (size 0.8) (drill 0.4) (layers "F.Cu" "B.Cu") (net 45))
-  (via (at 128.27 112.141) (size 0.8) (drill 0.4) (layers "F.Cu" "B.Cu") (net 45))
-  (segment (start 128.27 112.141) (end 128.27 118.491) (width 0.635) (layer "B.Cu") (net 45))
+  (segment (start 166.116 117.926) (end 166.116 119.507) (width 0.635) (layer "F.Cu") (net 44))
+  (segment (start 166.116 112.776) (end 166.116 111.252) (width 0.635) (layer "F.Cu") (net 44))
+  (via (at 166.116 111.252) (size 0.8) (drill 0.4) (layers "F.Cu" "B.Cu") (net 44))
+  (via (at 166.116 119.507) (size 0.8) (drill 0.4) (layers "F.Cu" "B.Cu") (net 44))
+  (segment (start 166.116 111.379) (end 166.116 119.507) (width 0.635) (layer "B.Cu") (net 44))
+  (segment (start 128.27 119.634) (end 128.27 112.268) (width 0.635) (layer "F.Cu") (net 45))
+  (segment (start 128.27 112.776) (end 128.27 111.252) (width 0.635) (layer "F.Cu") (net 45))
+  (segment (start 128.27 112.268) (end 128.27 112.776) (width 0.635) (layer "F.Cu") (net 45))
+  (segment (start 128.27 117.926) (end 128.27 119.634) (width 0.635) (layer "F.Cu") (net 45))
+  (via (at 128.27 119.634) (size 0.8) (drill 0.4) (layers "F.Cu" "B.Cu") (net 45))
+  (via (at 128.27 111.252) (size 0.8) (drill 0.4) (layers "F.Cu" "B.Cu") (net 45))
+  (segment (start 128.27 111.252) (end 128.27 119.634) (width 0.635) (layer "B.Cu") (net 45))
   (segment (start 121.92 112.776) (end 121.92 117.926) (width 0.635) (layer "F.Cu") (net 46))
-  (segment (start 121.92 112.776) (end 121.92 112.141) (width 0.635) (layer "F.Cu") (net 46))
-  (segment (start 121.92 118.491) (end 121.92 117.926) (width 0.635) (layer "F.Cu") (net 46))
-  (via (at 121.92 112.141) (size 0.8) (drill 0.4) (layers "F.Cu" "B.Cu") (net 46))
-  (via (at 121.92 118.491) (size 0.8) (drill 0.4) (layers "F.Cu" "B.Cu") (net 46))
-  (segment (start 121.92 112.141) (end 121.92 118.491) (width 0.635) (layer "B.Cu") (net 46))
+  (segment (start 121.92739 111.338411) (end 121.92 111.345801) (width 0.635) (layer "F.Cu") (net 46))
+  (segment (start 121.92 112.776) (end 121.92 111.25939) (width 0.635) (layer "F.Cu") (net 46))
+  (segment (start 121.92 111.25939) (end 121.92739 111.252) (width 0.635) (layer "F.Cu") (net 46))
+  (segment (start 121.92 117.926) (end 121.92 119.507) (width 0.635) (layer "F.Cu") (net 46))
+  (via (at 121.92739 111.252) (size 0.8) (drill 0.4) (layers "F.Cu" "B.Cu") (net 46))
+  (via (at 121.92 119.507) (size 0.8) (drill 0.4) (layers "F.Cu" "B.Cu") (net 46))
+  (segment (start 121.92739 111.338411) (end 121.92 111.345801) (width 0.635) (layer "B.Cu") (net 46))
+  (segment (start 121.92 111.345801) (end 121.92 119.507) (width 0.635) (layer "B.Cu") (net 46))
   (zone (net 43) (net_name "/Motor_1/OUT_1") (layers "F&B.Cu") (hatch edge 0.5)
     (priority 8)
@@
     (polygon
       (pts
-        (xy 171.831 111.633)
-        (xy 173.101 111.633)
+        (xy 171.831 110.49)
+        (xy 173.101 110.49)
         (xy 173.101 121.158)
         (xy 175.26 121.158)
@@
     (polygon
       (pts
-        (xy 165.481 111.633)
+        (xy 165.481 111.379)
         (xy 165.481 121.158)
         (xy 162.306 121.158)
@@
         (xy 167.005 121.031)
         (xy 166.751 121.031)
-        (xy 166.751 111.633)
+        (xy 166.751 111.379)
       )
     )
@@
     (polygon
       (pts
-        (xy 127.635 111.633)
-        (xy 128.905 111.633)
+        (xy 127.635 110.744)
+        (xy 128.905 110.744)
         (xy 128.905 121.285)
         (xy 131.572 121.285)
