File: tvca_controller/tvca_controller.kicad_pcb (KiCad board)
At the start: 2 copper layers, 84.3 x 59.2 mm, 57 parts, among them J1 Programming Header, J2 PT 1,5/ 4-5,0-H, J3 4DB-P108-02, J4 PT 1,5/ 4-5,0-H, J5 4DB-P108-02, J6 PT 1,5/ 4-5,0-H, J7 4DB-P108-02, J9 4DB-P108-02, U1 PIC18F26K83, U2 MCP2562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

Commit message: routing
Parts:
- moved D1 36.2 mm to (118.0, 91.0), turned to 180 degrees
- moved R9 31.3 mm to (123.2, 91.0), turned to 180 degrees
- moved C13 13.4 mm to (183.5, 116.7), turned to -90 degrees
- moved R14 13.4 mm to (159.1, 124.0), turned to -90 degrees
- moved C12 12.6 mm to (110.7, 92.1), turned to 90 degrees
- moved R10 9.14 mm to (161.1, 110.7)
- moved R17 7.69 mm to (135.5, 124.0), turned to -90 degrees
- moved C7 6.12 mm to (133.1, 112.3)
- moved R19 6.12 mm to (133.1, 118.4)
- moved R15 3.09 mm to (133.1, 116.8)
- moved R16 3.05 mm to (161.1, 119.9)
- moved U3 2.21 mm to (149.2, 102.7), turned to -90 degrees
- moved J5 1.02 mm to (165.7, 123.5)
- moved C8 0.54 mm to (166.5, 109.2)
- moved R11 0.51 mm to (133.1, 113.8)
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Connections:
- R9 pad 1: Net-(U1-RB5) -> Net-(U1-RA1)
- U1 pad 13: /CCW_1 -> /VBAT_2
- U1 pad 14: /CLW_1 -> /SEL_2
- U1 pad 17: /CLW_2 -> /SEL_1
- U1 pad 22: /VBAT_2 -> /CLW_1
- U1 pad 23: /VBAT_1 -> /CCW_1
- U1 pad 24: /SEL_2 -> /ENCDRA_1
- U1 pad 25: /SEL_1 -> /VBAT_1
- U1 pad 26: Net-(U1-RB5) -> /ENCDRB_1
- U1 pad 3: /ENCDRA_1 -> Net-(U1-RA1)
- U1 pad 4: /ENCDRB_1 -> /CLW_2
Routing:
- net +5V: track 0.00 -> 157.8 mm, vias 0 -> 3
- net /CUR_2: track 0.00 -> 73.2 mm, vias 0 -> 1
- net /CUR_1: track 0.00 -> 68.0 mm, vias 0 -> 1
- net /ENCDRB_2: track 0.00 -> 44.8 mm, vias 0 -> 1
- net /ENCDRA_1: track 0.00 -> 40.1 mm, vias 0 -> 1
- net /VBAT_2: track 0.00 -> 40.0 mm
- net /ENCDRA_2: track 0.00 -> 39.0 mm, vias 0 -> 1
- net /CUR_AMP: track 0.00 -> 36.7 mm, vias 0 -> 2
- net /ENCDRB_1: track 0.00 -> 34.7 mm, vias 0 -> 1
- net Net-(U8-CS): track 0.00 -> 34.1 mm, vias 0 -> 1
- net Net-(U9-CS): track 0.00 -> 32.9 mm, vias 0 -> 1
- net Net-(U8-IN_A): track 0.00 -> 27.6 mm, vias 0 -> 2
- net Net-(U9-SEL_0): track 0.00 -> 25.9 mm
- net Net-(U9-IN_B): track 0.00 -> 25.4 mm, vias 0 -> 2
- net Net-(U1-RA1): track 0.00 -> 23.8 mm, vias 0 -> 2
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