File: tvca_controller/motor.kicad_sch (KiCad schematic)
At the start: 18 parts, among them J3 4DB-P108-02, J4 PT 1,5/ 4-5,0-H, J5 4DB-P108-02, U8 VNH7070AS

Commit message: finish silkscreen
Parts:
- renumbered J4 to J3, J5 to J4, R7 to R10, R18 to R11, R5 to R4, R10 to R5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
