File: tvca_controller/tvca_controller.kicad_sch (KiCad schematic)
At the start: 21 parts, among them J1 Programming Header, J2 PT 1,5/ 4-5,0-H, U1 PIC18F26K83, U2 MCP2562, U3 INA180, Y1 Crystal 12 MHz

Commit message: finish silkscreen
Parts:
- renumbered C3 to C1, C1 to C2, C2 to C3, H3 to H2, H2 to H3, R9 to R1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
